File: aqua_driver.kicad_sch (KiCad schematic)
At the start: 9 parts, among them J1 HEATER IN, J2 230V IN, K1 FINDER-36.11, Q1 2N7000, U1 TCMT1100

Commit message: Fixed merge.
Parts:
- removed BT1: Battery_Cell, symbol Device:Battery_Cell
- removed C1: 100N, symbol Device:C
- removed J1: HEATER IN, symbol Connector_Generic:Conn_01x03
- removed J2: 230V IN, symbol Connector_Generic:Conn_01x03
- removed K1: FINDER-36.11, Relay_THT:Relay_SPDT_Finder_36.11, symbol Relay:FINDER-36.11
- removed Q1: 2N7000, Package_TO_SOT_THT:TO-92_Inline, symbol Transistor_FET:2N7000
- removed R1: R, symbol Device:R
- removed R2: 1K, symbol Device:R
- removed U1: TCMT1100, Package_SO:SOP-4_4.4x2.6mm_P1.27mm, symbol Isolator:TCMT1100
Connections:
- no-connect marks 1 -> 0
Other:
- note removed: "230V Connectors"
- note removed: "HEATER"

Commit message: Working on aqua_driver - temperature sensors.
Other:
- sheet Temperature control ports: added 1; removed none
Changed lines of the file:
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@@
       (effects (font (size 1.27 1.27)) (justify left top))
     )
+    (property "Footprint" "" (at 115.57 163.83 0)
+      (effects (font (size 1.27 1.27)) hide)
+    )
+    (property "Datasheet" "" (at 115.57 163.83 0)
+      (effects (font (size 1.27 1.27)) hide)
+    )
+    (pin "1")
     (instances
       (project "aqua_driver"
-        (path "/13f34ed6-0d14-48e4-b5f6-041bf4b3feac" (page "2"))
+        (path "/13f34ed6-0d14-48e4-b5f6-041bf4b3feac"
+          (reference "#PWR021") (unit 1)
+        )
       )
     )
