File: bluetooth_module.kicad_sch (KiCad schematic)
At the start: 0 parts

Commit message: Place bluetooth module with basic connectivity
Parts:
- added U10: RN4871, RF_Module:Microchip_RN4871, symbol RF_Bluetooth:RN4871
Connections:
- new net BT_IND: U10.15 (P2_7)
- new net BT_RX: U10.7 (UART_RX)
- new net BT_TX: U10.8 (UART_TX)
- new net GND: U10.13 (GND), U10.2 (GND)
Changed lines of the file:
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@@
 (kicad_sch (version 20230121) (generator eeschema)
   (paper "A4")
+  (junction (at 135.89 107.95) (diameter 0) (color 0 0 0 0)
+  )
+  (wire (pts (xy 100.33 78.74) (xy 118.11 78.74))
+    (stroke (width 0) (type default))
+  )
+  (wire (pts (xy 153.67 93.98) (xy 172.72 93.98))
+    (stroke (width 0) (type default))
+  )
+  (wire (pts (xy 135.89 107.95) (xy 135.89 110.49))
+    (stroke (width 0) (type default))
+  )
+  (wire (pts (xy 133.35 101.6) (xy 133.35 107.95))
+    (stroke (width 0) (type default))
+  )
+  (wire (pts (xy 133.35 107.95) (xy 135.89 107.95))
+    (stroke (width 0) (type default))
+  )
+  (wire (pts (xy 135.89 107.95) (xy 138.43 107.95))
+    (stroke (width 0) (type default))
+  )
+  (wire (pts (xy 100.33 81.28) (xy 118.11 81.28))
+    (stroke (width 0) (type default))
+  )
+  (wire (pts (xy 138.43 107.95) (xy 138.43 101.6))
+    (stroke (width 0) (type default))
+  )
+  (hierarchical_label "BT_IND" (shape output) (at 172.72 93.98 0) (fields_autoplaced)
+    (effects (font (size 1.27 1.27)) (justify left))
+  )
+  (hierarchical_label "BT_RX" (shape input) (at 100.33 78.74 180) (fields_autoplaced)
+    (effects (font (size 1.27 1.27)) (justify right))
+  )
+  (hierarchical_label "BT_TX" (shape output) (at 100.33 81.28 180) (fields_autoplaced)
+    (effects (font (size 1.27 1.27)) (justify right))
+  )
+  (symbol (lib_id "RF_Bluetooth:RN4871") (at 135.89 86.36 0) (unit 1)
+    (in_bom yes) (on_board yes) (dnp no) (fields_autoplaced)
+    (property "Reference" "U10" (at 138.0841 68.58 0)
+      (effects (font (size 1.27 1.27)) (justify left))
+    )
+    (property "Value" "RN4871" (at 138.0841 71.12 0)
+      (effects (font (size 1.27 1.27)) (justify left))
+    )
+    (property "Footprint" "RF_Module:Microchip_RN4871" (at 135.89 104.14 0)
+      (effects (font (size 1.27 1.27)) hide)
+    )
+    (property "Datasheet" "http://ww1.microchip.com/downloads/en/DeviceDoc/50002489A.pdf" (at 123.19 72.39 0)
+      (effects (font (size 1.27 1.27)) hide)
+    )
+    (pin "7")
+    (pin "14")
+    (pin "15")
+    (pin "16")
+    (pin "9")
+    (pin "1")
+    (pin "8")
+    (pin "6")
+    (pin "4")
+    (pin "2")
+    (pin "13")
+    (pin "12")
+    (pin "3")
+    (pin "11")
+    (pin "10")
+    (pin "5")
+    (instances
+      (project "aqua_driver"
+        (path "/13f34ed6-0d14-48e4-b5f6-041bf4b3feac"
+          (reference "U10") (unit 1)
+        )
+        (path "/13f34ed6-0d14-48e4-b5f6-041bf4b3feac/c2b58e3c-fd64-47de-8341-9bd2a4eed71c"
+          (reference "U10") (unit 1)
+        )
+      )
+    )
+  )
+  (symbol (lib_id "power:GND") (at 135.89 110.49 0) (unit 1)
+    (in_bom yes) (on_board yes) (dnp no) (fields_autoplaced)
+    (property "Reference" "#PWR01" (at 135.89 116.84 0)
+      (effects (font (size 1.27 1.27)) hide)
+    )
+    (property "Value" "GND" (at 135.89 115.57 0)
+      (effects (font (size 1.27 1.27)))
+    )
+    (property "Footprint" "" (at 135.89 110.49 0)
+      (effects (font (size 1.27 1.27)) hide)
+    )
+    (property "Datasheet" "" (at 135.89 110.49 0)
+      (effects (font (size 1.27 1.27)) hide)
+    )
+    (pin "1")
+    (instances
+      (project "aqua_driver"
+        (path "/13f34ed6-0d14-48e4-b5f6-041bf4b3feac/c2b58e3c-fd64-47de-8341-9bd2a4eed71c"
+          (reference "#PWR01") (unit 1)
+        )
+      )
+    )
+  )
 )
